Commit message: upload

File: universal_robot/ur_description/urdf/common.gazebo.xacro (robot description, xacro)
@@ -21,35 +21,3 @@
 -->
   </gazebo>
-   <!-- camera_link -->
-  <gazebo reference="camera_link">
-    <mu1>0.2</mu1>
-    <mu2>0.2</mu2>
-    <material>Gazebo/Green</material>
-  </gazebo>
-  <!--camera-->
-  <gazebo reference="camera_link">
-    <sensor type="camera" name="camera1">
-      <update_rate>30.0</update_rate>
-      <camera name="head">
-        <horizontal_fov>1.3962634</horizontal_fov>
-        <image>
-          <width>800</width>
-          <height>800</height>
-          <format>R8G8B8</format>
-        </image>
-        <clip>
-          <near>0.02</near>
-          <far>300</far>
-        </clip>
-        <noise>
-          <type>gaussian</type>
-          <!-- Noise is sampled independently per pixel on each frame.
-               That pixel's noise value is added to each of its color
-               channels, which at that point lie in the range [0,1]. -->
-          <mean>0.0</mean>
-          <stddev>0.007</stddev>
-        </noise>
-      </camera>
-    </sensor>
-  </gazebo>
 </robot>

File: universal_robot/ur_description/urdf/ur3_joint_limited_robot.urdf.xacro (robot description, xacro)
@@ -9,11 +9,10 @@
   <!-- arm -->
   <xacro:ur3_robot prefix="" joint_limited="true"
-    shoulder_pan_lower_limit="${-pi}" shoulder_pan_upper_limit="${pi}"
-    shoulder_lift_lower_limit="${-pi}" shoulder_lift_upper_limit="${pi}"
-    elbow_joint_lower_limit="${-pi}" elbow_joint_upper_limit="${pi}"
-    wrist_1_lower_limit="${-pi}" wrist_1_upper_limit="${pi}"
-    wrist_2_lower_limit="${-pi}" wrist_2_upper_limit="${pi}"
-    wrist_3_lower_limit="${-pi}" wrist_3_upper_limit="${pi}"
-    transmission_hw_interface="$(arg transmission_hw_interface)"
+    shoulder_pan_lower_limit="${-4*pi}" shoulder_pan_upper_limit="${4*pi}"
+    shoulder_lift_lower_limit="${-4*pi}" shoulder_lift_upper_limit="${4*pi}"
+    elbow_joint_lower_limit="${-4*pi}" elbow_joint_upper_limit="${4*pi}"
+    wrist_1_lower_limit="${-4*pi}" wrist_1_upper_limit="${4*pi}"
+    wrist_2_lower_limit="${-4*pi}" wrist_2_upper_limit="${4*pi}"
+    wrist_3_lower_limit="${-4*pi}" wrist_3_upper_limit="${4*pi}"
   />
   <link name="world" />
